File: KiCad/keyboard.kicad_pcb (KiCad board)
At the start: 2 copper layers, 154 parts

Commit message: pushing everything cuz i'm lazy, will cull later
Parts:
- removed L?: LED, footprints:CHERRY_MX_LED
- removed REF**: TO-220, Power_Integrations:TO-220
- removed S0:5/6, S0:7/8: MX, footprints:CHERRY_PCB_200H
- added C1: 1uF, Capacitors_SMD:C_0805_HandSoldering, B.Cu at (142.5, 62.5)
- added C2: 1uF, Capacitors_SMD:C_0805_HandSoldering, B.Cu at (140.0, 25.0)
- added C3: 0.1uF, Capacitors_SMD:C_0805_HandSoldering, B.Cu at (160.5, 56.0)
- added C6: 0.1uF, Capacitors_SMD:C_0805_HandSoldering, B.Cu at (140.0, 27.0)
- added C7: 1uF, Capacitors_SMD:C_0805_HandSoldering, B.Cu at (142.5, 64.5)
- added C8: 10pF, Capacitors_SMD:C_0805_HandSoldering, B.Cu at (119.0, 52.5)
- added C9: 10pF, Capacitors_SMD:C_0805_HandSoldering, B.Cu at (119.0, 50.5)
- added R5: 1k, Resistors_SMD:R_0805_HandSoldering, B.Cu at (155.0, 44.5)
- added R_CAPS1: RESISTOR, Resistors_SMD:R_0805_HandSoldering, B.Cu at (273.0, 102.0)
- added R_FN1: RESISTOR, Resistors_SMD:R_0805_HandSoldering, B.Cu at (83.5, 102.0)
- C4, C5: renamed from REF**; value C_0805_HandSoldering -> 0.1uF
- Crystal1: renamed from REF**; value ABM3 -> 16MHz
- D0:0, D0:1, D0:10, D0:11, D0:12, D0:13, D0:2, D0:3, D0:4, D0:5, D0:6, D0:7, D0:8, D0:9, D1:0, D1:1, D1:10, D1:11, D1:12, D1:13, D1:2, D1:3, D1:4, D1:5, D1:6, D1:7, D1:8, D1:9, D2:0, D2:1, D2:10, D2:11, D2:12, D2:13, D2:2, D2:3, D2:4, D2:5, D2:6, D2:7, D2:8, D2:9, D3:0, D3:1, D3:10, D3:11, D3:12, D3:13, D3:2, D3:3, D3:4, D3:5, D3:6, D3:7, D3:8, D3:9, D4:0, D4:1, D4:10, D4:11, D4:12, D4:13, D4:2, D4:3, D4:4, D4:5, D4:6, D4:7, D4:8, D4:9: value Diode_DO-35_SOD27_Horizontal_RM10 -> DIODE
- P1: renamed from REF**; value USB_Mini-B -> USB_OTG
- R3, R4: value R_0805_HandSoldering -> 22
- S0:0, S0:1, S0:10, S0:11, S0:12, S0:13, S0:2, S0:3, S0:4, S0:5, S0:6, S0:7, S0:8, S0:9, S1:0, S1:1, S1:10, S1:11, S1:12, S1:13, S1:2, S1:3, S1:4, S1:5, S1:6, S1:7, S1:8, S1:9, S2:0, S2:1, S2:10, S2:11, S2:12, S2:13, S2:2, S2:3, S2:4, S2:5, S2:6, S2:7, S2:8, S2:9, S3:0, S3:1, S3:10, S3:11, S3:12, S3:13, S3:2, S3:3, S3:4, S3:5, S3:6, S3:7, S3:8, S3:9, S4:0, S4:1, S4:10, S4:11, S4:12, S4:13, S4:2, S4:3, S4:4, S4:5, S4:6, S4:7, S4:8, S4:9: value MX -> SWITCH_PUSH
- S_RST1: renamed from REF**; value SW_SPST_PTS645 -> SW_PUSH
- U2: renamed from REF**; value MLF-44_Atmel -> ATmega32U4
- moved S_RST1 68.6 mm to (117.0, 66.2)
- moved Crystal1 50.6 mm to (114.5, 52.5), turned to 270 degrees
- moved D3:9 15.0 mm to (185.0, 31.0), turned to 270 degrees
- moved D2:7 13.9 mm to (152.0, 68.0), turned to 0 degrees
- moved D2:6 13.5 mm to (141.0, 68.0), turned to 180 degrees
- moved D3:10 10.7 mm to (203.9, 35.8), turned to 270 degrees
- moved D3:4 10.2 mm to (106.2, 35.8), turned to 270 degrees
- moved D4:7 10.2 mm to (163.2, 16.8), turned to 270 degrees
- moved D4:10 10.2 mm to (203.9, 16.8), turned to 270 degrees
- moved D4:11 10.2 mm to (223.0, 16.8), turned to 270 degrees
- moved D4:8 10.2 mm to (166.0, 16.8), turned to 270 degrees
- moved D4:9 10.2 mm to (185.0, 16.8), turned to 270 degrees
- moved D3:3 10.2 mm to (87.0, 35.8), turned to 270 degrees
- moved D3:7 10.2 mm to (163.2, 35.8), turned to 270 degrees
- moved D4:13 10.2 mm to (261.0, 16.9), turned to 270 degrees
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- gave numbers to parts that had none: 2
Connections:
- C4 pad 1: (no net) -> Net-(C1-Pad1)
- C4 pad 2: (no net) -> GND
- C5 pad 1: (no net) -> Net-(C1-Pad1)
- C5 pad 2: (no net) -> GND
- Crystal1 pad 1: (no net) -> Net-(C9-Pad1)
- Crystal1 pad 2: (no net) -> Net-(C8-Pad1)
- D0:0 pad 1: (no net) -> Net-(D0:0-Pad1)
- D0:0 pad 2: (no net) -> /COL0
- D0:1 pad 1: (no net) -> Net-(D0:1-Pad1)
- D0:1 pad 2: (no net) -> /COL1
- D0:10 pad 1: (no net) -> Net-(D0:10-Pad1)
- D0:10 pad 2: (no net) -> /COL10
- D0:11 pad 1: (no net) -> Net-(D0:11-Pad1)
- D0:11 pad 2: (no net) -> /COL11
- D0:12 pad 1: (no net) -> Net-(D0:12-Pad1)
- D0:12 pad 2: (no net) -> /COL12
- D0:13 pad 1: (no net) -> Net-(D0:13-Pad1)
- D0:13 pad 2: (no net) -> /COL13
- D0:2 pad 1: (no net) -> Net-(D0:2-Pad1)
- D0:2 pad 2: (no net) -> /COL2
- D0:3 pad 1: (no net) -> Net-(D0:3-Pad1)
- D0:3 pad 2: (no net) -> /COL3
- D0:4 pad 1: (no net) -> Net-(D0:4-Pad1)
- D0:4 pad 2: (no net) -> /COL4
- D0:5 pad 1: (no net) -> Net-(D0:5-Pad1)
- D0:5 pad 2: (no net) -> /COL5
- D0:6 pad 1: (no net) -> Net-(D0:6-Pad1)
- D0:6 pad 2: (no net) -> /COL6
- D0:7 pad 1: (no net) -> Net-(D0:7-Pad1)
- D0:7 pad 2: (no net) -> /COL7
- D0:8 pad 1: (no net) -> Net-(D0:8-Pad1)
- D0:8 pad 2: (no net) -> /COL8
- D0:9 pad 1: (no net) -> Net-(D0:9-Pad1)
- D0:9 pad 2: (no net) -> /COL9
- D1:0 pad 1: (no net) -> Net-(D1:0-Pad1)
- D1:0 pad 2: (no net) -> /COL0
- D1:1 pad 1: (no net) -> Net-(D1:1-Pad1)
- D1:1 pad 2: (no net) -> /COL1
- D1:10 pad 1: (no net) -> Net-(D1:10-Pad1)
- D1:10 pad 2: (no net) -> /COL10
- D1:11 pad 1: (no net) -> Net-(D1:11-Pad1)
- D1:11 pad 2: (no net) -> /COL11
- D1:12 pad 1: (no net) -> Net-(D1:12-Pad1)
- D1:12 pad 2: (no net) -> /COL12
- D1:13 pad 1: (no net) -> Net-(D1:13-Pad1)
- D1:13 pad 2: (no net) -> /COL13
- D1:2 pad 1: (no net) -> Net-(D1:2-Pad1)
- D1:2 pad 2: (no net) -> /COL2
- D1:3 pad 1: (no net) -> Net-(D1:3-Pad1)
- D1:3 pad 2: (no net) -> /COL3
- D1:4 pad 1: (no net) -> Net-(D1:4-Pad1)
- D1:4 pad 2: (no net) -> /COL4
- D1:5 pad 1: (no net) -> Net-(D1:5-Pad1)
- D1:5 pad 2: (no net) -> /COL5
- D1:6 pad 1: (no net) -> Net-(D1:6-Pad1)
- D1:6 pad 2: (no net) -> /COL6
- D1:7 pad 1: (no net) -> Net-(D1:7-Pad1)
- D1:7 pad 2: (no net) -> /COL7
- D1:8 pad 1: (no net) -> Net-(D1:8-Pad1)
- D1:8 pad 2: (no net) -> /COL8
- D1:9 pad 1: (no net) -> Net-(D1:9-Pad1)
- D1:9 pad 2: (no net) -> /COL9
- D2:0 pad 1: (no net) -> Net-(D2:0-Pad1)
- D2:0 pad 2: (no net) -> /COL0
- D2:1 pad 1: (no net) -> Net-(D2:1-Pad1)
- D2:1 pad 2: (no net) -> /COL1
- D2:10 pad 1: (no net) -> Net-(D2:10-Pad1)
- D2:10 pad 2: (no net) -> /COL10
- D2:11 pad 1: (no net) -> Net-(D2:11-Pad1)
- D2:11 pad 2: (no net) -> /COL11
- D2:12 pad 1: (no net) -> Net-(D2:12-Pad1)
- D2:12 pad 2: (no net) -> /COL12
- D2:13 pad 1: (no net) -> Net-(D2:13-Pad1)
- D2:13 pad 2: (no net) -> /COL13
- D2:2 pad 1: (no net) -> Net-(D2:2-Pad1)
- D2:2 pad 2: (no net) -> /COL2
- D2:3 pad 1: (no net) -> Net-(D2:3-Pad1)
- D2:3 pad 2: (no net) -> /COL3
- D2:4 pad 1: (no net) -> Net-(D2:4-Pad1)
- D2:4 pad 2: (no net) -> /COL4
- D2:5 pad 1: (no net) -> Net-(D2:5-Pad1)
- D2:5 pad 2: (no net) -> /COL5
- D2:6 pad 1: (no net) -> Net-(D2:6-Pad1)
- D2:6 pad 2: (no net) -> /COL6
- D2:7 pad 1: (no net) -> Net-(D2:7-Pad1)
- D2:7 pad 2: (no net) -> /COL7
- D2:8 pad 1: (no net) -> Net-(D2:8-Pad1)
- D2:8 pad 2: (no net) -> /COL8
- D2:9 pad 1: (no net) -> Net-(D2:9-Pad1)
- D2:9 pad 2: (no net) -> /COL9
- D3:0 pad 1: (no net) -> Net-(D3:0-Pad1)
- D3:0 pad 2: (no net) -> /COL0
- D3:1 pad 1: (no net) -> Net-(D3:1-Pad1)
- D3:1 pad 2: (no net) -> /COL1
- D3:10 pad 1: (no net) -> Net-(D3:10-Pad1)
- D3:10 pad 2: (no net) -> /COL10
- D3:11 pad 1: (no net) -> Net-(D3:11-Pad1)
- D3:11 pad 2: (no net) -> /COL11
- D3:12 pad 1: (no net) -> Net-(D3:12-Pad1)
- D3:12 pad 2: (no net) -> /COL12
- D3:13 pad 1: (no net) -> Net-(D3:13-Pad1)
- D3:13 pad 2: (no net) -> /COL13
- D3:2 pad 1: (no net) -> Net-(D3:2-Pad1)
- D3:2 pad 2: (no net) -> /COL2
- D3:3 pad 1: (no net) -> Net-(D3:3-Pad1)
- D3:3 pad 2: (no net) -> /COL3
- D3:4 pad 1: (no net) -> Net-(D3:4-Pad1)
- D3:4 pad 2: (no net) -> /COL4
- D3:5 pad 1: (no net) -> Net-(D3:5-Pad1)
- D3:5 pad 2: (no net) -> /COL5
- D3:6 pad 1: (no net) -> Net-(D3:6-Pad1)
- D3:6 pad 2: (no net) -> /COL6
- D3:7 pad 1: (no net) -> Net-(D3:7-Pad1)
- D3:7 pad 2: (no net) -> /COL7
- D3:8 pad 1: (no net) -> Net-(D3:8-Pad1)
- D3:8 pad 2: (no net) -> /COL8
- D3:9 pad 1: (no net) -> Net-(D3:9-Pad1)
- D3:9 pad 2: (no net) -> /COL9
- D4:0 pad 1: (no net) -> Net-(D4:0-Pad1)
- D4:0 pad 2: (no net) -> /COL0
- D4:1 pad 1: (no net) -> Net-(D4:1-Pad1)
- D4:1 pad 2: (no net) -> /COL1
- D4:10 pad 1: (no net) -> Net-(D4:10-Pad1)
- D4:10 pad 2: (no net) -> /COL10
- D4:11 pad 1: (no net) -> Net-(D4:11-Pad1)
- D4:11 pad 2: (no net) -> /COL11
- D4:12 pad 1: (no net) -> Net-(D4:12-Pad1)
- D4:12 pad 2: (no net) -> /COL12
- D4:13 pad 1: (no net) -> Net-(D4:13-Pad1)
- D4:13 pad 2: (no net) -> /COL13
- D4:2 pad 1: (no net) -> Net-(D4:2-Pad1)
- D4:2 pad 2: (no net) -> /COL2
- D4:3 pad 1: (no net) -> Net-(D4:3-Pad1)
- D4:3 pad 2: (no net) -> /COL3
- D4:4 pad 1: (no net) -> Net-(D4:4-Pad1)
- D4:4 pad 2: (no net) -> /COL4
- D4:5 pad 1: (no net) -> Net-(D4:5-Pad1)
- D4:5 pad 2: (no net) -> /COL5
- D4:6 pad 1: (no net) -> Net-(D4:6-Pad1)
- D4:6 pad 2: (no net) -> /COL6
- D4:7 pad 1: (no net) -> Net-(D4:7-Pad1)
- D4:7 pad 2: (no net) -> /COL7
- D4:8 pad 1: (no net) -> Net-(D4:8-Pad1)
- D4:8 pad 2: (no net) -> /COL8
- D4:9 pad 1: (no net) -> Net-(D4:9-Pad1)
- D4:9 pad 2: (no net) -> /COL9
- D_CAPS1 pad 1: (no net) -> GND
- D_CAPS1 pad 2: (no net) -> Net-(D_CAPS1-Pad2)
- D_FN1 pad 1: (no net) -> GND
- D_FN1 pad 2: (no net) -> Net-(D_FN1-Pad2)
- P1 pad 1: (no net) -> Net-(C1-Pad1)
- P1 pad 2: (no net) -> Net-(P1-Pad2)
- P1 pad 3: (no net) -> Net-(P1-Pad3)
- P1 pad 4: (no net) -> Net-(P1-Pad4)
- P1 pad 5: (no net) -> GND
- P1 pad 6: (no net) -> GND
- R3 pad 1: (no net) -> Net-(P1-Pad2)
- R3 pad 2: (no net) -> Net-(R3-Pad2)
- R4 pad 1: (no net) -> Net-(P1-Pad3)
- R4 pad 2: (no net) -> Net-(R4-Pad2)
- S0:0 pad 1: (no net) -> /ROW0
- S0:0 pad 2: (no net) -> Net-(D0:0-Pad1)
- S0:1 pad 1: (no net) -> /ROW0
- S0:1 pad 2: (no net) -> Net-(D0:1-Pad1)
- S0:10 pad 1: (no net) -> /ROW0
- S0:10 pad 2: (no net) -> Net-(D0:10-Pad1)
- S0:11 pad 1: (no net) -> /ROW0
- S0:11 pad 2: (no net) -> Net-(D0:11-Pad1)
- S0:12 pad 1: (no net) -> /ROW0
- S0:12 pad 2: (no net) -> Net-(D0:12-Pad1)
- S0:13 pad 1: (no net) -> /ROW0
- S0:13 pad 2: (no net) -> Net-(D0:13-Pad1)
- S0:2 pad 1: (no net) -> /ROW0
- S0:2 pad 2: (no net) -> Net-(D0:2-Pad1)
- S0:3 pad 1: (no net) -> /ROW0
- S0:3 pad 2: (no net) -> Net-(D0:3-Pad1)
- S0:4 pad 1: (no net) -> /ROW0
- S0:4 pad 2: (no net) -> Net-(D0:4-Pad1)
- S0:5 pad 1: (no net) -> Net-(S0:5-Pad1)
- S0:5 pad 2: (no net) -> Net-(D0:5-Pad1)
- S0:6 pad 1: (no net) -> /ROW0
- S0:6 pad 2: (no net) -> Net-(D0:6-Pad1)
- S0:7 pad 1: (no net) -> /ROW0
- S0:7 pad 2: (no net) -> Net-(D0:7-Pad1)
- S0:8 pad 1: (no net) -> /ROW0
- S0:8 pad 2: (no net) -> Net-(D0:8-Pad1)
- S0:9 pad 1: (no net) -> /ROW0
- S0:9 pad 2: (no net) -> Net-(D0:9-Pad1)
- S1:0 pad 1: (no net) -> /ROW1
- S1:0 pad 2: (no net) -> Net-(D1:0-Pad1)
- S1:1 pad 1: (no net) -> /ROW1
- S1:1 pad 2: (no net) -> Net-(D1:1-Pad1)
- S1:10 pad 1: (no net) -> /ROW1
- S1:10 pad 2: (no net) -> Net-(D1:10-Pad1)
- S1:11 pad 1: (no net) -> /ROW1
- S1:11 pad 2: (no net) -> Net-(D1:11-Pad1)
- S1:12 pad 1: (no net) -> /ROW1
- S1:12 pad 2: (no net) -> Net-(D1:12-Pad1)
- S1:13 pad 1: (no net) -> /ROW1
- S1:13 pad 2: (no net) -> Net-(D1:13-Pad1)
- S1:2 pad 1: (no net) -> /ROW1
- S1:2 pad 2: (no net) -> Net-(D1:2-Pad1)
- S1:3 pad 1: (no net) -> /ROW1
- S1:3 pad 2: (no net) -> Net-(D1:3-Pad1)
- S1:4 pad 1: (no net) -> /ROW1
- S1:4 pad 2: (no net) -> Net-(D1:4-Pad1)
- S1:5 pad 1: (no net) -> /ROW1
- S1:5 pad 2: (no net) -> Net-(D1:5-Pad1)
- S1:6 pad 1: (no net) -> /ROW1
- S1:6 pad 2: (no net) -> Net-(D1:6-Pad1)
- S1:7 pad 1: (no net) -> /ROW1
- S1:7 pad 2: (no net) -> Net-(D1:7-Pad1)
- S1:8 pad 1: (no net) -> /ROW1
- S1:8 pad 2: (no net) -> Net-(D1:8-Pad1)
- S1:9 pad 1: (no net) -> /ROW1
- S1:9 pad 2: (no net) -> Net-(D1:9-Pad1)
- S2:0 pad 1: (no net) -> /ROW2
- S2:0 pad 2: (no net) -> Net-(D2:0-Pad1)
- S2:1 pad 1: (no net) -> /ROW2
- S2:1 pad 2: (no net) -> Net-(D2:1-Pad1)
- S2:10 pad 1: (no net) -> /ROW2
- S2:10 pad 2: (no net) -> Net-(D2:10-Pad1)
- S2:11 pad 1: (no net) -> /ROW2
- S2:11 pad 2: (no net) -> Net-(D2:11-Pad1)
- S2:12 pad 1: (no net) -> /ROW2
- S2:12 pad 2: (no net) -> Net-(D2:12-Pad1)
- S2:13 pad 1: (no net) -> /ROW2
- S2:13 pad 2: (no net) -> Net-(D2:13-Pad1)
- S2:2 pad 1: (no net) -> /ROW2
- S2:2 pad 2: (no net) -> Net-(D2:2-Pad1)
- S2:3 pad 1: (no net) -> /ROW2
- S2:3 pad 2: (no net) -> Net-(D2:3-Pad1)
- S2:4 pad 1: (no net) -> /ROW2
- S2:4 pad 2: (no net) -> Net-(D2:4-Pad1)
- S2:5 pad 1: (no net) -> /ROW2
- S2:5 pad 2: (no net) -> Net-(D2:5-Pad1)
- S2:6 pad 1: (no net) -> /ROW2
- S2:6 pad 2: (no net) -> Net-(D2:6-Pad1)
- S2:7 pad 1: (no net) -> /ROW2
- S2:7 pad 2: (no net) -> Net-(D2:7-Pad1)
- S2:8 pad 1: (no net) -> /ROW2
- S2:8 pad 2: (no net) -> Net-(D2:8-Pad1)
- S2:9 pad 1: (no net) -> /ROW2
- S2:9 pad 2: (no net) -> Net-(D2:9-Pad1)
- S3:0 pad 1: (no net) -> /ROW3
- S3:0 pad 2: (no net) -> Net-(D3:0-Pad1)
- S3:1 pad 1: (no net) -> /ROW3
- S3:1 pad 2: (no net) -> Net-(D3:1-Pad1)
- S3:10 pad 1: (no net) -> /ROW3
- S3:10 pad 2: (no net) -> Net-(D3:10-Pad1)
- S3:11 pad 1: (no net) -> /ROW3
- S3:11 pad 2: (no net) -> Net-(D3:11-Pad1)
- S3:12 pad 1: (no net) -> /ROW3
- S3:12 pad 2: (no net) -> Net-(D3:12-Pad1)
- S3:13 pad 1: (no net) -> /ROW3
- S3:13 pad 2: (no net) -> Net-(D3:13-Pad1)
- S3:2 pad 1: (no net) -> /ROW3
- S3:2 pad 2: (no net) -> Net-(D3:2-Pad1)
- S3:3 pad 1: (no net) -> /ROW3
- S3:3 pad 2: (no net) -> Net-(D3:3-Pad1)
- S3:4 pad 1: (no net) -> /ROW3
- S3:4 pad 2: (no net) -> Net-(D3:4-Pad1)
- S3:5 pad 1: (no net) -> /ROW3
- S3:5 pad 2: (no net) -> Net-(D3:5-Pad1)
- S3:6 pad 1: (no net) -> /ROW3
- S3:6 pad 2: (no net) -> Net-(D3:6-Pad1)
- S3:7 pad 1: (no net) -> /ROW3
- S3:7 pad 2: (no net) -> Net-(D3:7-Pad1)
- S3:8 pad 1: (no net) -> /ROW3
- S3:8 pad 2: (no net) -> Net-(D3:8-Pad1)
- S3:9 pad 1: (no net) -> /ROW3
- S3:9 pad 2: (no net) -> Net-(D3:9-Pad1)
- S4:0 pad 1: (no net) -> /ROW4
- S4:0 pad 2: (no net) -> Net-(D4:0-Pad1)
- S4:1 pad 1: (no net) -> /ROW4
- S4:1 pad 2: (no net) -> Net-(D4:1-Pad1)
- S4:10 pad 1: (no net) -> /ROW4
- S4:10 pad 2: (no net) -> Net-(D4:10-Pad1)
- S4:11 pad 1: (no net) -> /ROW4
- S4:11 pad 2: (no net) -> Net-(D4:11-Pad1)
- S4:12 pad 1: (no net) -> /ROW4
- S4:12 pad 2: (no net) -> Net-(D4:12-Pad1)
- S4:13 pad 1: (no net) -> /ROW4
- S4:13 pad 2: (no net) -> Net-(D4:13-Pad1)
- S4:2 pad 1: (no net) -> /ROW4
- S4:2 pad 2: (no net) -> Net-(D4:2-Pad1)
- S4:3 pad 1: (no net) -> /ROW4
- S4:3 pad 2: (no net) -> Net-(D4:3-Pad1)
- S4:4 pad 1: (no net) -> /ROW4
- S4:4 pad 2: (no net) -> Net-(D4:4-Pad1)
- S4:5 pad 1: (no net) -> /ROW4
- S4:5 pad 2: (no net) -> Net-(D4:5-Pad1)
- S4:6 pad 1: (no net) -> /ROW4
- S4:6 pad 2: (no net) -> Net-(D4:6-Pad1)
- S4:7 pad 1: (no net) -> /ROW4
- S4:7 pad 2: (no net) -> Net-(D4:7-Pad1)
- S4:8 pad 1: (no net) -> /ROW4
- S4:8 pad 2: (no net) -> Net-(D4:8-Pad1)
- S4:9 pad 1: (no net) -> /ROW4
- S4:9 pad 2: (no net) -> Net-(D4:9-Pad1)
- S_RST1 pad 1: (no net) -> GND
- S_RST1 pad 2: (no net) -> Net-(S_RST1-Pad2)
- U2 pad 1: (no net) -> /E6
- U2 pad 10: (no net) -> /ROW2
- U2 pad 11: (no net) -> /ROW3
- U2 pad 12: (no net) -> /B7
- U2 pad 13: (no net) -> Net-(S_RST1-Pad2)
- U2 pad 14: (no net) -> Net-(C1-Pad1)
- U2 pad 15: (no net) -> GND
- U2 pad 16: (no net) -> Net-(C8-Pad1)
- U2 pad 17: (no net) -> Net-(C9-Pad1)
- U2 pad 18: (no net) -> /COL0
- U2 pad 19: (no net) -> /COL1
- U2 pad 2: (no net) -> Net-(C1-Pad1)
- U2 pad 20: (no net) -> /COL2
- U2 pad 21: (no net) -> /COL3
- U2 pad 22: (no net) -> /COL5
- U2 pad 23: (no net) -> GND
- U2 pad 24: (no net) -> Net-(C1-Pad1)
- U2 pad 25: (no net) -> /COL4
- U2 pad 26: (no net) -> /COL6
- U2 pad 27: (no net) -> /COL7
- U2 pad 28: (no net) -> /ROW4
- U2 pad 29: (no net) -> /LED_FN
- U2 pad 3: (no net) -> Net-(R3-Pad2)
- U2 pad 30: (no net) -> /LED_CAPS
- U2 pad 31: (no net) -> /C6
- U2 pad 32: (no net) -> /C7
- U2 pad 33: (no net) -> Net-(R5-Pad2)
- U2 pad 34: (no net) -> Net-(C1-Pad1)
- U2 pad 35: (no net) -> GND
- U2 pad 36: (no net) -> /COL13
- U2 pad 37: (no net) -> /COL12
- U2 pad 38: (no net) -> /COL11
- U2 pad 39: (no net) -> /COL10
- U2 pad 4: (no net) -> Net-(R4-Pad2)
- U2 pad 40: (no net) -> /COL9
- U2 pad 41: (no net) -> /COL8
- U2 pad 42: (no net) -> Net-(C3-Pad1)
- U2 pad 43: (no net) -> GND
- U2 pad 44: (no net) -> Net-(C1-Pad1)
- U2 pad 5: (no net) -> GND
- U2 pad 6: (no net) -> Net-(C7-Pad1)
- U2 pad 7: (no net) -> Net-(C1-Pad1)
- U2 pad 8: (no net) -> /ROW0
- U2 pad 9: (no net) -> /ROW1
Routing:
- net GND: track 0.00 -> 542.9 mm, vias 0 -> 18
- net /ROW0: track 0.00 -> 308.2 mm, vias 0 -> 2
- net /ROW4: track 0.00 -> 296.4 mm, vias 0 -> 2
- net /ROW1: track 0.00 -> 285.1 mm
- net /ROW3: track 0.00 -> 280.6 mm, vias 0 -> 2
- net /ROW2: track 0.00 -> 268.1 mm, vias 0 -> 1
- net /COL0: track 0.00 -> 199.1 mm, vias 0 -> 4
- net /COL13: track 0.00 -> 196.2 mm, vias 0 -> 2
- net /LED_CAPS: track 0.00 -> 185.6 mm, vias 0 -> 2
- net /COL1: track 0.00 -> 178.2 mm
- net /COL12: track 0.00 -> 176.4 mm, vias 0 -> 2
- net /COL2: track 0.00 -> 158.8 mm
- net /COL11: track 0.00 -> 157.3 mm, vias 0 -> 2
- net /COL3: track 0.00 -> 138.9 mm
- net /COL10: track 0.00 -> 137.8 mm, vias 0 -> 2
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Other:
- net class Default: clearance 0.2 -> 0.1524; trace_width 0.25 -> 0.1524; via_dia 0.6 -> 0.635
- rule trace_clearance: 0.2 -> 0.1524
- rule trace_min: 0.2 -> 0.1524
- rule via_min_size: 0.4 -> 0.381

Commit message: culling old materiasl and backup files
Routing:
- net Net-(C1-Pad1): track 127.8 -> 116.4 mm, vias 6 -> 8
- net GND: track 542.9 -> 540.7 mm, vias 18 -> 16
- net /COL13: track 196.2 -> 197.8 mm
- net /COL9: track 119.7 -> 119.1 mm, vias 3 -> 1
- net /COL10: track 137.8 -> 137.5 mm, vias 2 -> 0
- net /COL11: track 157.3 -> 157.0 mm, vias 2 -> 0
- net /COL12: track 176.4 -> 176.5 mm, vias 2 -> 0
