File: KiCad/keyboard.kicad_pcb (KiCad board)
At the start: 2 copper layers, 265 x 94 mm, 239 parts, among them J1 USBMINI_B05, M1 MountingHole_4mm, M2 MountingHole_4mm, M3 MountingHole_4mm, M4 MountingHole_4mm, T1 CONN_1, T2 CONN_1, T3 CONN_1, T4 CONN_1, U1 ATmega32U4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

Commit message: submitting quote for case and cover
Parts:
- M1, M2, M3, M4: value MountingHole_4mm -> MountingHole_6.4mm; footprint Mounting_Holes:MountingHole_4mm -> Mounting_Holes:MountingHole_6.4mm_M6
- moved L_PWR1 1.17 mm to (250.6, 79.2)
- moved J1 0.30 mm to (212.5, 60.5)
- moved M3 0.25 mm to (117.2, 117.3)
- moved M2 0.25 mm to (307.8, 98.2)
- moved M4 0.17 mm to (155.3, 79.2)
- moved M1 0.17 mm to (269.6, 136.3)
Routing:
- net /led/lcol12: track 183.1 -> 185.2 mm
- net /matrix/col12: track 180.0 -> 181.8 mm
- net /led/lcol11: track 171.9 -> 170.2 mm
- net /matrix/col13: track 207.8 -> 208.8 mm
- net Net-(L1:0-Pad1): track 270.6 -> 271.5 mm
- net /led/lcol10: track 150.5 -> 151.2 mm, vias 4 -> 2
- net Net-(L2:0-Pad1): track 276.3 -> 276.9 mm
- net /matrix/col10: track 146.1 -> 146.7 mm
