File: KiCad/keyboard.sch (KiCad schematic (older format))
At the start: 167 parts

Commit message: pushing everything cuz i'm lazy, will cull later
Parts:
- removed D0:5/6, D0:7/8: DIODE, symbol DIODE
- removed R1, R2: 0, symbol RESISTOR
- removed S0:5/6, S0:7/8: SWITCH_PUSH, symbol SWITCH_PUSH
- removed U?: MCP1825, symbol MCP1825
- gave numbers to parts that had none: 3
- renumbered Crystal to Crystal1, D3:4 to D3:3, D_CAPS to D_CAPS1, D_FN to D_FN1, R4 to R5, R_CAPS to R_CAPS1, R_FN to R_FN1, S_RST to S_RST1
Connections:
- net GND: now also P1.6 (shield)
- net ROW0: no longer S0:5.1
- net at C2.1, C4.1, C5.1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: now also C1.1, P1.1 (VCC), U2.2 (UVCC), U2.7 (VBUS)
Changed lines of the file:
@@
 LIBS:contrib
 LIBS:valves
-LIBS:components
 LIBS:cherry
 LIBS:mcp1825
@@
 $EndComp
 $Comp
-L DIODE D3:4
+L DIODE D3:3
 U 1 1 56AB5FB2
 P 4800 6700
-F 0 "D3:4" H 4700 6650 40  0000 C CNN
+F 0 "D3:3" H 4700 6650 40  0000 C CNN
 F 1 "DIODE" H 4800 6750 40  0000 C CNN
 F 2 "" H 4800 6700 60  0000 C CNN
@@
 $EndComp
 $Comp
-L DIODE D?
+L DIODE D3:4
 U 1 1 56AB5FB8
 P 5550 6700
-F 0 "D?" H 5450 6650 40  0000 C CNN
+F 0 "D3:4" H 5450 6650 40  0000 C CNN
 F 1 "DIODE" H 5550 6750 40  0000 C CNN
 F 2 "" H 5550 6700 60  0000 C CNN
@@
 $EndComp
 $Comp
-L RESISTOR R_CAPS
+L RESISTOR R_CAPS1
 U 1 1 56AC73C4
 P 12000 8950
-F 0 "R_CAPS" V 12000 8850 50  0000 C CNN
+F 0 "R_CAPS1" V 12000 8850 50  0000 C CNN
 F 1 "RESISTOR" V 12000 9050 50  0000 C CNN
 F 2 "" H 12000 8950 60  0000 C CNN
@@
 $EndComp
 $Comp
-L RESISTOR R_FN
+L RESISTOR R_FN1
 U 1 1 56AC7E58
 P 4500 9000
-F 0 "R_FN" V 4500 8900 50  0000 C CNN
+F 0 "R_FN1" V 4500 8900 50  0000 C CNN
 F 1 "RESISTOR" V 4500 9100 50  0000 C CNN
 F 2 "" H 4500 9000 60  0000 C CNN
@@
 $EndComp
 $Comp
-L LED D_FN
+L LED D_FN1
 U 1 1 56ACF314
 P 4950 9000
-F 0 "D_FN" H 4950 9100 50  0000 C CNN
+F 0 "D_FN1" H 4950 9100 50  0000 C CNN
 F 1 "LED" H 4950 8900 50  0000 C CNN
 F 2 "" H 4950 9000 50  0000 C CNN
@@
 $EndComp
 $Comp
-L LED D_CAPS
+L LED D_CAPS1
 U 1 1 56ACF608
 P 12450 8950
-F 0 "D_CAPS" V 12450 9050 50  0000 C CNN
+F 0 "D_CAPS1" V 12450 9050 50  0000 C CNN
 F 1 "LED" H 12450 8850 50  0000 C CNN
 F 2 "" H 12450 8950 50  0000 C CNN
@@
 $EndComp
 $Comp
-L ATmega32U4 U?
+L ATmega32U4 U2
 U 1 1 56AD4506
 P 7650 2350
-F 0 "U?" H 6750 4050 50  0000 C CNN
+F 0 "U2" H 6750 4050 50  0000 C CNN
 F 1 "ATmega32U4" H 7000 800 50  0000 C CNN
 F 2 "" H 8850 3450 50  0000 C CNN
@@
 $EndComp
 $Comp
-L USB_OTG P?
+L USB_OTG P1
 U 1 1 56B6DAED
 P 2800 2500
-F 0 "P?" H 3125 2375 50  0000 C CNN
+F 0 "P1" H 3125 2375 50  0000 C CNN
 F 1 "USB_OTG" H 2800 2700 50  0000 C CNN
 F 2 "" V 2750 2400 50  0000 C CNN
@@
 $EndComp
 $Comp
-L SWITCH_PUSH S0:5/6
-U 1 1 56B20287
-P 6000 9400
-F 0 "S0:5/6" H 6150 9510 50  0000 C CNN
-F 1 "SWITCH_PUSH" H 6000 9320 50  0000 C CNN
-F 2 "" H 6000 9400 60  0000 C CNN
-F 3 "" H 6000 9400 60  0000 C CNN
-	1    6000 9400
-	1    0    0    -1
-$EndComp
-$Comp
-L DIODE D0:5/6
-U 1 1 56B2028D
-P 6300 9200
-F 0 "D0:5/6" H 6200 9150 40  0000 C CNN
-F 1 "DIODE" H 6300 9250 40  0000 C CNN
-F 2 "" H 6300 9200 60  0000 C CNN
-F 3 "" H 6300 9200 60  0000 C CNN
-	1    6300 9200
-	0    -1   -1   0
-$EndComp
-$Comp
-L SWITCH_PUSH S0:7/8
-U 1 1 56B21E2C
-P 7500 9400
-F 0 "S0:7/8" H 7650 9510 50  0000 C CNN
-F 1 "SWITCH_PUSH" H 7500 9320 50  0000 C CNN
-F 2 "" H 7500 9400 60  0000 C CNN
-F 3 "" H 7500 9400 60  0000 C CNN
-	1    7500 9400
-	1    0    0    -1
-$EndComp
-$Comp
-L DIODE D0:7/8
-U 1 1 56B21E32
-P 7800 9200
-F 0 "D0:7/8" H 7700 9150 40  0000 C CNN
-F 1 "DIODE" H 7800 9250 40  0000 C CNN
-F 2 "" H 7800 9200 60  0000 C CNN
-F 3 "" H 7800 9200 60  0000 C CNN
-	1    7800 9200
-	0    -1   -1   0
-$EndComp
-$Comp
-L MCP1825 U?
-U 1 1 56B308E4
-P 3600 1400
-F 0 "U?" H 3600 1600 60  0000 C CNN
-F 1 "MCP1825" H 3600 1500 60  0000 C CNN
-F 2 "" H 3600 1400 60  0000 C CNN
-F 3 "" H 3600 1400 60  0000 C CNN
-	1    3600 1400
-	1    0    0    -1
-$EndComp
-$Comp
 L CP1 C1
 U 1 1 56B44CCB
@@
 $EndComp
 $Comp
-L GND #PWR?
+L GND #PWR03
 U 1 1 56B44F94
 P 3050 1100
-F 0 "#PWR?" H 3050 850 50  0001 C CNN
+F 0 "#PWR03" H 3050 850 50  0001 C CNN
 F 1 "GND" H 3050 950 50  0000 C CNN
 F 2 "" H 3050 1100 50  0000 C CNN
@@
 $EndComp
 $Comp
-L Crystal Crystal
+L Crystal Crystal1
 U 1 1 56B4B3EC
 P 5050 3900
-F 0 "Crystal" H 5050 4050 50  0000 C CNN
+F 0 "Crystal1" H 5050 4050 50  0000 C CNN
 F 1 "16MHz" H 5050 3750 50  0000 C CNN
 F 2 "" H 5050 3900 50  0000 C CNN
@@
 $EndComp
 $Comp
-L GND #PWR?
+L GND #PWR04
 U 1 1 56B502F4
 P 4750 4400
-F 0 "#PWR?" H 4750 4150 50  0001 C CNN
+F 0 "#PWR04" H 4750 4150 50  0001 C CNN
 F 1 "GND" H 4750 4250 50  0000 C CNN
 F 2 "" H 4750 4400 50  0000 C CNN
@@
 $EndComp
 $Comp
-L GND #PWR?
+L GND #PWR05
 U 1 1 56B504DC
 P 5300 4400
-F 0 "#PWR?" H 5300 4150 50  0001 C CNN
+F 0 "#PWR05" H 5300 4150 50  0001 C CNN
 F 1 "GND" H 5300 4250 50  0000 C CNN
 F 2 "" H 5300 4400 50  0000 C CNN
@@
 $EndComp
 $Comp
-L GND #PWR?
+L GND #PWR06
 U 1 1 56B5A272
 P 4200 2150
-F 0 "#PWR?" H 4200 1900 50  0001 C CNN
+F 0 "#PWR06" H 4200 1900 50  0001 C CNN
 F 1 "GND" H 4200 2000 50  0000 C CNN
 F 2 "" H 4200 2150 50  0000 C CNN
@@
 $EndComp
 $Comp
-L GND #PWR?
+L GND #PWR07
 U 1 1 56B5CADF
 P 3350 2800
-F 0 "#PWR?" H 3350 2550 50  0001 C CNN
+F 0 "#PWR07" H 3350 2550 50  0001 C CNN
 F 1 "GND" H 3350 2650 50  0000 C CNN
 F 2 "" H 3350 2800 50  0000 C CNN
@@
 $EndComp
 Wire Wire Line
-	7900 5650 7900 9000
+	7900 5650 7900 8350
 Wire Wire Line
 	7800 7750 7900 7750
@@
 	6400 7750 6300 7750
 Wire Wire Line
-	6400 5650 6400 9000
-Wire Wire Line
 	6400 8350 6300 8350
 Connection ~ 1950 6400
@@
 	4950 8900 4950 8750
 Connection ~ 5700 8900
-Wire Wire Line
-	5700 8750 5700 9400
 Connection ~ 7200 8900
 Wire Wire Line
-	7200 8750 7200 9400
+	7200 8900 7200 8750
 Connection ~ 8700 8900
 Wire Wire Line
@@
 Connection ~ 11650 7750
 Wire Wire Line
-	6400 9000 6300 9000
-Connection ~ 6400 8350
-Wire Wire Line
 	6450 8750 6450 8900
 Connection ~ 6450 8900
@@
 	8650 8350 8550 8350
 Connection ~ 8650 7750
-Wire Wire Line
-	7900 9000 7800 9000
 Connection ~ 7900 8350
 Wire Wire Line
@@
 	4200 1800 4200 1850
 Wire Wire Line
-	3100 2700 3600 2700
-Wire Wire Line
 	3350 2700 3350 2800
 Wire Wire Line
@@
 	3050 600  3050 800
 Connection ~ 3050 600
-Wire Wire Line
-	3600 2700 3600 1750
 Connection ~ 3350 2700
 Wire Wire Line
 	3300 1850 3300 2300
 Wire Wire Line
-	3050 1850 3050 1400
-Wire Wire Line
-	3050 1400 3250 1400
-Connection ~ 3050 1850
-Wire Wire Line
-	3950 1300 3950 1400
-$Comp
-L RESISTOR R1
-U 1 1 56B68195
-P 4200 1550
-F 0 "R1" V 4200 1450 50  0000 C CNN
-F 1 "0" V 4200 1650 50  0000 C CNN
-F 2 "" H 4200 1550 60  0000 C CNN
-F 3 "" H 4200 1550 60  0000 C CNN
-	1    4200 1550
-	1    0    0    -1
-$EndComp
-$Comp
-L RESISTOR R2
-U 1 1 56B6DEDE
-P 4200 1050
-F 0 "R2" V 4200 950 50  0000 C CNN
-F 1 "0" V 4200 1150 50  0000 C CNN
-F 2 "" H 4200 1050 60  0000 C CNN
-F 3 "" H 4200 1050 60  0000 C CNN
-	1    4200 1050
-	1    0    0    -1
-$EndComp
-Wire Wire Line
-	3950 1300 6400 1300
-Connection ~ 4200 1300
-Wire Wire Line
-	4200 800  4200 600
-Connection ~ 4200 600
-Wire Wire Line
-	6050 900  6050 1300
+	6050 1300 6050 900
 Wire Wire Line
 	6050 900  6400 900
@@
 Connection ~ 6050 1000
 $Comp
-L GND #PWR?
+L GND #PWR08
 U 1 1 56B9C199
 P 5000 850
-F 0 "#PWR?" H 5000 600 50  0001 C CNN
+F 0 "#PWR08" H 5000 600 50  0001 C CNN
 F 1 "GND" H 5000 700 50  0000 C CNN
 F 2 "" H 5000 850 50  0000 C CNN
@@
 Connection ~ 6050 1300
 $Comp
-L GND #PWR?
+L GND #PWR09
 U 1 1 56BBD318
 P 6300 3800
-F 0 "#PWR?" H 6300 3550 50  0001 C CNN
+F 0 "#PWR09" H 6300 3550 50  0001 C CNN
 F 1 "GND" H 6300 3650 50  0000 C CNN
 F 2 "" H 6300 3800 50  0000 C CNN
@@
 	5300 2900 6400 2900
 Wire Wire Line
-	5800 1300 5800 1300
+	4650 1300 6400 1300
 Wire Wire Line
 	5800 2100 5800 1300
@@
 $EndComp
 $Comp
-L GND #PWR?
+L GND #PWR010
 U 1 1 56BDBD72
 P 5150 2500
-F 0 "#PWR?" H 5150 2250 50  0001 C CNN
+F 0 "#PWR010" H 5150 2250 50  0001 C CNN
 F 1 "GND" H 5150 2350 50  0000 C CNN
 F 2 "" H 5150 2500 50  0000 C CNN
@@
 $EndComp
 $Comp
-L GND #PWR?
+L GND #PWR011
 U 1 1 56BDBF6C
 P 5350 2500
-F 0 "#PWR?" H 5350 2250 50  0001 C CNN
+F 0 "#PWR011" H 5350 2250 50  0001 C CNN
 F 1 "GND" H 5350 2350 50  0000 C CNN
 F 2 "" H 5350 2500 50  0000 C CNN
@@
 $EndComp
 $Comp
-L GND #PWR?
+L GND #PWR012
 U 1 1 56BDC166
 P 5550 2500
-F 0 "#PWR?" H 5550 2250 50  0001 C CNN
+F 0 "#PWR012" H 5550 2250 50  0001 C CNN
 F 1 "GND" H 5550 2350 50  0000 C CNN
 F 2 "" H 5550 2500 50  0000 C CNN
@@
 $EndComp
 $Comp
-L SW_PUSH S_RST
+L SW_PUSH S_RST1
 U 1 1 56BE5E2B
 P 6100 2200
-F 0 "S_RST" H 6250 2310 50  0000 C CNN
+F 0 "S_RST1" H 6250 2310 50  0000 C CNN
 F 1 "SW_PUSH" H 6100 2120 50  0000 C CNN
 F 2 "" H 6100 2200 50  0000 C CNN
@@
 	8850 1800 9400 1800
 $Comp
-L RESISTOR R4
+L RESISTOR R5
 U 1 1 56C22707
 P 9200 2900
-F 0 "R4" V 9200 2800 50  0000 C CNN
+F 0 "R5" V 9200 2800 50  0000 C CNN
 F 1 "1k" V 9200 3000 50  0000 C CNN
 F 2 "" H 9200 2900 60  0000 C CNN
@@
 $EndComp
 $Comp
-L GND #PWR?
+L GND #PWR013
 U 1 1 56C229BA
 P 9450 2900
-F 0 "#PWR?" H 9450 2650 50  0001 C CNN
+F 0 "#PWR013" H 9450 2650 50  0001 C CNN
 F 1 "GND" H 9450 2750 50  0000 C CNN
 F 2 "" H 9450 2900 50  0000 C CNN
@@
 Text Label 9400 3000 0    60   ~ 0
 E6
+Wire Wire Line
+	6400 5650 6400 8350
+Wire Wire Line
+	4650 1300 4650 600
+Connection ~ 4650 600
+Wire Wire Line
+	3100 2700 3350 2700
+Wire Wire Line
+	2700 2900 3200 2900
+Wire Wire Line
+	3200 2900 3200 2700
+Connection ~ 3200 2700
 $EndSCHEMATC

Commit message: updated to fix some errors
Connections:
- net ROW0: now also S0:5.1
Other:
- moved on the sheet: C2, C3, D_FN1
Changed lines of the file:
@@
 L LED D_FN1
 U 1 1 56ACF314
-P 4950 9000
-F 0 "D_FN1" H 4950 9100 50  0000 C CNN
-F 1 "LED" H 4950 8900 50  0000 C CNN
-F 2 "" H 4950 9000 50  0000 C CNN
-F 3 "" H 4950 9000 50  0000 C CNN
-	1    4950 9000
+P 5050 9000
+F 0 "D_FN1" H 5050 9100 50  0000 C CNN
+F 1 "LED" H 5050 8900 50  0000 C CNN
+F 2 "" H 5050 9000 50  0000 C CNN
+F 3 "" H 5050 9000 50  0000 C CNN
+	1    5050 9000
 	-1   0    0    1
 $EndComp
@@
 L GND #PWR01
 U 1 1 56B4D623
-P 5150 9000
-F 0 "#PWR01" H 5150 8750 50  0001 C CNN
-F 1 "GND" H 5150 8850 50  0000 C CNN
-F 2 "" H 5150 9000 50  0000 C CNN
-F 3 "" H 5150 9000 50  0000 C CNN
-	1    5150 9000
+P 5250 9000
+F 0 "#PWR01" H 5250 8750 50  0001 C CNN
+F 1 "GND" H 5250 8850 50  0000 C CNN
+F 2 "" H 5250 9000 50  0000 C CNN
+F 3 "" H 5250 9000 50  0000 C CNN
+	1    5250 9000
 	0    -1   -1   0
 $EndComp
@@
 	1    0    0    -1
 $EndComp
-$Comp
-L GND #PWR07
-U 1 1 56B5CADF
-P 3350 2800
-F 0 "#PWR07" H 3350 2550 50  0001 C CNN
-F 1 "GND" H 3350 2650 50  0000 C CNN
-F 2 "" H 3350 2800 50  0000 C CNN
-F 3 "" H 3350 2800 50  0000 C CNN
-	1    3350 2800
-	1    0    0    -1
-$EndComp
 Wire Wire Line
 	7900 5650 7900 8350
@@
 	4200 1800 4200 1850
 Wire Wire Line
-	3350 2700 3350 2800
-Wire Wire Line
 	3100 2300 3300 2300
 Wire Wire Line
@@
 	3050 600  3050 800
 Connection ~ 3050 600
-Connection ~ 3350 2700
 Wire Wire Line
 	3300 1850 3300 2300
@@
 Connection ~ 6050 1000
 $Comp
-L GND #PWR08
+L GND #PWR07
 U 1 1 56B9C199
-P 5000 850
-F 0 "#PWR08" H 5000 600 50  0001 C CNN
-F 1 "GND" H 5000 700 50  0000 C CNN
-F 2 "" H 5000 850 50  0000 C CNN
-F 3 "" H 5000 850 50  0000 C CNN
-	1    5000 850
+P 5200 800
+F 0 "#PWR07" H 5200 550 50  0001 C CNN
+F 1 "GND" H 5200 650 50  0000 C CNN
+F 2 "" H 5200 800 50  0000 C CNN
+F 3 "" H 5200 800 50  0000 C CNN
+	1    5200 800
 	-1   0    0    1
 $EndComp
@@
 L CP1 C2
 U 1 1 56B9C387
-P 5000 1000
-F 0 "C2" H 5025 1100 50  0000 L CNN
-F 1 "1uF" H 5025 900 50  0000 L CNN
-F 2 "" H 5000 1000 50  0000 C CNN
-F 3 "" H 5000 1000 50  0000 C CNN
-	1    5000 1000
+P 5200 950
+F 0 "C2" H 5225 1050 50  0000 L CNN
+F 1 "1uF" H 5225 850 50  0000 L CNN
+F 2 "" H 5200 950 50  0000 C CNN
+F 3 "" H 5200 950 50  0000 C CNN
+	1    5200 950
 	-1   0    0    1
 $EndComp
 Wire Wire Line
-	5000 1300 5000 1150
+	5000 1100 5000 1300
 Connection ~ 5000 1300
 Wire Wire Line
@@
 Connection ~ 6050 1300
 $Comp
-L GND #PWR09
+L GND #PWR08
 U 1 1 56BBD318
-P 6300 3800
-F 0 "#PWR09" H 6300 3550 50  0001 C CNN
-F 1 "GND" H 6300 3650 50  0000 C CNN
-F 2 "" H 6300 3800 50  0000 C CNN
-F 3 "" H 6300 3800 50  0000 C CNN
-	1    6300 3800
+P 6300 3850
+F 0 "#PWR08" H 6300 3600 50  0001 C CNN
+F 1 "GND" H 6300 3700 50  0000 C CNN
+F 2 "" H 6300 3850 50  0000 C CNN
+F 3 "" H 6300 3850 50  0000 C CNN
+	1    6300 3850
 	1    0    0    -1
 $EndComp
@@
 	6300 3700 6400 3700
 Wire Wire Line
-	6300 1900 6300 3800
+	6300 1900 6300 3850
 Wire Wire Line
 	6400 3600 6300 3600
@@
 Connection ~ 6300 3600
 Wire Wire Line
-	6400 3400 6300 3400
+	5800 3400 6400 3400
 Connection ~ 6300 3500
 Wire Wire Line
@@
 $EndComp
 $Comp
-L GND #PWR010
+L GND #PWR09
 U 1 1 56BDBD72
 P 5150 2500
-F 0 "#PWR010" H 5150 2250 50  0001 C CNN
+F 0 "#PWR09" H 5150 2250 50  0001 C CNN
 F 1 "GND" H 5150 2350 50  0000 C CNN
 F 2 "" H 5150 2500 50  0000 C CNN
@@
 $EndComp
 $Comp
-L GND #PWR011
+L GND #PWR010
 U 1 1 56BDBF6C
 P 5350 2500
-F 0 "#PWR011" H 5350 2250 50  0001 C CNN
+F 0 "#PWR010" H 5350 2250 50  0001 C CNN
 F 1 "GND" H 5350 2350 50  0000 C CNN
 F 2 "" H 5350 2500 50  0000 C CNN
@@
 $EndComp
 $Comp
-L GND #PWR012
+L GND #PWR011
 U 1 1 56BDC166
 P 5550 2500
-F 0 "#PWR012" H 5550 2250 50  0001 C CNN
+F 0 "#PWR011" H 5550 2250 50  0001 C CNN
 F 1 "GND" H 5550 2350 50  0000 C CNN
 F 2 "" H 5550 2500 50  0000 C CNN
@@
 $EndComp
 $Comp
-L GND #PWR013
+L GND #PWR012
 U 1 1 56C229BA
 P 9450 2900
-F 0 "#PWR013" H 9450 2650 50  0001 C CNN
+F 0 "#PWR012" H 9450 2650 50  0001 C CNN
 F 1 "GND" H 9450 2750 50  0000 C CNN
 F 2 "" H 9450 2900 50  0000 C CNN
@@
 	6400 1200 5700 1200
 Wire Wire Line
-	5700 1200 5700 1050
+	5700 1200 5700 950
 $Comp
 L CP1 C3
 U 1 1 56C3D1B1
-P 5700 900
-F 0 "C3" H 5725 1000 50  0000 L CNN
-F 1 "0.1uF" H 5725 800 50  0000 L CNN
-F 2 "" H 5700 900 50  0000 C CNN
-F 3 "" H 5700 900 50  0000 C CNN
-	1    5700 900
+P 5700 800
+F 0 "C3" H 5725 900 50  0000 L CNN
+F 1 "0.1uF" H 5725 700 50  0000 L CNN
+F 2 "" H 5700 800 50  0000 C CNN
+F 3 "" H 5700 800 50  0000 C CNN
+	1    5700 800
 	-1   0    0    1
 $EndComp
 Wire Wire Line
-	5700 750  5700 600
-Text Label 5700 600  0    60   ~ 0
+	5700 650  6000 650
+Text Label 6000 650  0    60   ~ 0
 AREF
 Text Label 9400 1500 0    60   ~ 0
@@
 Connection ~ 4650 600
 Wire Wire Line
-	3100 2700 3350 2700
-Wire Wire Line
 	2700 2900 3200 2900
 Wire Wire Line
 	3200 2900 3200 2700
 Connection ~ 3200 2700
+Wire Wire Line
+	5200 1100 5000 1100
+Wire Wire Line
+	5700 8900 5700 8750
+Wire Wire Line
+	3100 2700 5800 2700
+Wire Wire Line
+	5800 2700 5800 3400
+Wire Wire Line
+	4850 9000 4750 9000
 $EndSCHEMATC
