File: KiCad/keyboard-MIT.kicad_pcb (KiCad board)
At the start: 2 copper layers, 268.3 x 98.3 mm, 156 parts, among them P1 USB_OTG, U2 ATmega32U4

Commit message: separating the different layouts
Parts:
- added H1: MountingHole_2.2mm_M2, Mounting_Holes:MountingHole_2.2mm_M2, F.Cu at (240.5, 50.5)
- added H1: MountingHole_2.2mm_M2, Mounting_Holes:MountingHole_2.2mm_M2, F.Cu at (202.5, 88.5)
- added H1: MountingHole_2.2mm_M2, Mounting_Holes:MountingHole_2.2mm_M2, F.Cu at (88.5, 31.5)
- added H1: MountingHole_2.2mm_M2, Mounting_Holes:MountingHole_2.2mm_M2, F.Cu at (50.5, 69.5)
- S0:5/6, S0:7/8: footprint footprints:CHERRY_PCB_200H -> footprints.pretty:CHERRY_PCB_200H_U
- moved D2:7 17.7 mm to (163.5, 54.5), turned to 270 degrees
- moved C5 9.64 mm to (140.0, 31.1), turned to 180 degrees
- moved R_CAPS1 9.15 mm to (263.9, 101.8)
- moved C7 8.57 mm to (151.0, 65.8), turned to 0 degrees
- moved C1 8.51 mm to (151.0, 63.0), turned to 0 degrees
- moved C4 7.78 mm to (140.0, 29.1), turned to 180 degrees
- moved R3 5.15 mm to (144.8, 25.9)
- moved R4 5.15 mm to (146.8, 25.9)
- moved C3 4.27 mm to (164.7, 57.0), turned to 0 degrees
- moved P1 2.30 mm to (146.0, 13.3)
- moved R5 1.91 mm to (154.2, 46.2)
- moved R_FN1 0.42 mm to (83.2, 101.7)
- turned S0:5/6 to 180 degrees
- turned S0:7/8 to 180 degrees
Routing:
- net GND: track 530.2 -> 444.1 mm, vias 18 -> 4
- net Net-(C1-Pad1): track 116.4 -> 69.6 mm, vias 8 -> 0
- net /ROW4: track 296.4 -> 322.8 mm, vias 2 -> 0
- net /ROW2: track 268.1 -> 293.1 mm
- net /COL4: track 124.1 -> 145.2 mm, vias 0 -> 1
- net /COL10: track 137.5 -> 116.9 mm
- net /COL3: track 138.9 -> 118.8 mm
- net /COL12: track 176.5 -> 156.8 mm
- net /COL7: track 109.2 -> 128.6 mm
- net /LED_FN: track 128.9 -> 148.0 mm, vias 6 -> 4
- net Net-(P1-Pad3): track 24.1 -> 8.10 mm, vias 2 -> 0
- net /LED_CAPS: track 185.6 -> 170.1 mm
- net /COL6: track 108.7 -> 122.8 mm, vias 1 -> 2
- net Net-(D3:9-Pad1): track 17.4 -> 9.39 mm, vias 1 -> 0
- net Net-(R3-Pad2): track 33.7 -> 40.6 mm
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Other:
- board size 268.3 x 98.3 mm -> 260 x 94.1 mm
