File: KiCad/prototype_keyboard.kicad_pcb (KiCad board)
At the start: 2 copper layers, 265 x 94 mm, 176 parts, among them J1 USBMINI_B05, M1 MountingHole_2.5mm, M2 MountingHole_2.5mm, M3 MountingHole_2.5mm, M4 MountingHole_2.5mm, P1 CONN_1, P2 CONN_1, P3 CONN_1, P4 CONN_1, U1 ATmega32U4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

Commit message: big update, got quote :(
Parts:
- removed D0:6, D0:8: D, Diodes_SMD:SOD-123
- removed S0:5, S0:6, S0:7, S0:8: SW_PUSH, footprints:CHERRY_PCB_100H
- removed S0:6/7: SW_PUSH, .pretty:CHERRY_PCB_400H
- C4: value 0.1uF -> 1uF
- C6: value 1uF -> 0.1uF
- J1: footprint usb_ports:USB_MINI-B_MOLEX_54819-0519 -> .pretty:USB_MINI-B_MOLEX_54819-0519-hole
- L_PWR1: footprint LEDs:LED_0805 -> LEDs:LED-3MM
- R1: moved to B.Cu
- moved R1 112.5 mm to (84.5, 112.0), turned to 90 degrees
- moved D4:7 8.05 mm to (218.8, 72.8), turned to 90 degrees
- moved R7 1.60 mm to (246.0, 80.2)
- moved L_PWR1 1.25 mm to (250.5, 78.0)
- moved G*** 0.33 mm to (202.8, 116.8)
- moved J1 0.25 mm to (212.2, 58.5)
Routing:
- net /LED_CAPS2: track 13.5 -> 139.4 mm, vias 1 -> 2
- net Net-(L_CAPS2-Pad2): track 124.3 -> 3.28 mm, vias 1 -> 0
- net Net-(D0:6-Pad2): track 22.5 -> 0.00 mm
- net /COL8: track 96.5 -> 77.5 mm
- net /COL6: track 90.4 -> 71.4 mm
- net Net-(D0:8-Pad2): track 12.7 -> 0.00 mm
- net /COL7: track 96.2 -> 84.8 mm
- net Net-(J1-Pad2): track 10.7 -> 8.13 mm
- net /ROW0: track 324.9 -> 323.0 mm, vias 0 -> 1
- net Net-(L_PWR1-Pad2): track 1.96 -> 3.69 mm
- net Net-(D4:7-Pad2): track 2.45 -> 4.14 mm
- net /LED_PWR: track 43.7 -> 42.1 mm
- net GND: track 162.5 -> 161.0 mm
- net VCC: track 73.1 -> 73.8 mm
Other:
- net class Default: via_drill 0.34 -> 0.4
