File: KiCad/prototype_keyboard.sch (KiCad schematic (older format))
At the start: 171 parts, among them J1 USBMINI_B05, P1 CONN_1, P2 CONN_1, P3 CONN_1, P4 CONN_1, U1 ATmega32U4, X1 CRYSTAL(4pin)

Commit message: big update, got quote :(
Parts:
- removed D0:6, D0:8: D, symbol D
- removed S0:5, S0:6, S0:6/7, S0:7, S0:8: SW_PUSH, symbol SW_PUSH
- renumbered C6 to C4, C4 to C5, C5 to C6
