File: KiCad/keyboard-rev3.sch (KiCad schematic (older format))
At the start: 22 parts, among them J1 USBMINI_B05, T1 CONN_1, T2 CONN_1, T3 CONN_1, T4 CONN_1, U1 ATmega32U4, X1 CRYSTAL(4pin)

Commit message: making revisions
Changed lines of the file:
@@
 LIBS:contrib
 LIBS:valves
+LIBS:components
 LIBS:keyboard-cache
 EELAYER 25 0
@@
 U 58D5B17B
 F0 "matrix" 60
-F1 "matrix.sch" 60
+F1 "matrix-rev3.sch" 60
 F2 "row4" T L 8050 2250 60
 F3 "row1" T L 8050 1950 60
@@
 U 58D595A8
 F0 "led" 60
-F1 "led.sch" 60
+F1 "led-rev3.sch" 60
 F2 "~reset~" T L 2900 5500 60
 F3 "mosi" T L 2900 5200 60
