File: KiCad/keyboard-rev3.kicad_pcb (KiCad board)
At the start: 2 copper layers, 265 x 94 mm, 239 parts, among them J1 USBMINI_B05, M1 MountingHole_4mm, M2 MountingHole_4mm, M3 MountingHole_4mm, M4 MountingHole_4mm, T1 CONN_1, T2 CONN_1, T3 CONN_1, T4 CONN_1, U1 ATmega32U4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

Commit message: making revisions
Parts:
- added D0:6: D, lib:SOD-123D, B.Cu at (197.8, 137.5)
- added D0:8: D, lib:SOD-123D, B.Cu at (235.7, 138.3)
- added L0:5: LED, lib:CHERRY_MX_LED, F.Cu at (183.9, 145.8)
- added L0:5-6.5: LED, lib:CHERRY_MX_LED, F.Cu at (188.7, 145.8)
- added L0:6: LED, lib:CHERRY_MX_LED, F.Cu at (203.0, 145.8)
- added L0:6.5: LED, lib:CHERRY_MX_LED, F.Cu at (212.5, 145.8)
- added L0:6.5-8: LED, lib:CHERRY_MX_LED, F.Cu at (236.3, 145.9)
- added L0:7: LED, lib:CHERRY_MX_LED, F.Cu at (222.0, 145.8)
- added L0:8: LED, lib:CHERRY_MX_LED, F.Cu at (241.1, 145.8)
- added S0:4-9: SW_PUSH, lib:CHERRY_PCB_600H, F.Cu at (212.4, 145.9)
- added S0:5: SW_PUSH, lib:CHERRY_PCB_100H, F.Cu at (183.9, 145.8)
- added S0:5-6.5: SW_PUSH, lib:CHERRY_PCB_150H, F.Cu at (188.7, 145.8)
- added S0:5-8: SW_PUSH, lib:CHERRY_PCB_400H, F.Cu at (212.5, 145.8)
- added S0:6: SW_PUSH, lib:CHERRY_PCB_100H, F.Cu at (203.0, 145.8)
- added S0:6.5: SW_PUSH, lib:CHERRY_PCB_100H, F.Cu at (212.5, 145.9)
- added S0:6.5-8: SW_PUSH, lib:CHERRY_PCB_150H, F.Cu at (236.3, 145.8)
- added S0:7: SW_PUSH, lib:CHERRY_PCB_100H, F.Cu at (222.0, 145.8)
- added S0:8: SW_PUSH, lib:CHERRY_PCB_100H, F.Cu at (241.1, 145.8)
- moved L0:7/8 0.16 mm to (231.6, 145.9)
- moved S0:7/8 0.16 mm to (231.6, 145.9)
- moved L0:5/6 0.13 mm to (193.5, 145.8)
- moved S0:5/6 0.13 mm to (193.5, 145.8)
Routing:
- net /led/lcol11: track 171.9 -> 122.8 mm
- net /led/lcol8: track 100.0 -> 66.3 mm, vias 2 -> 0
- net Net-(L0:0-Pad1): track 277.7 -> 307.4 mm, vias 1 -> 2
- net Net-(D0:6-Pad2): track 0.00 -> 26.9 mm, vias 0 -> 2
- net /led/lcol6: track 85.5 -> 110.2 mm, vias 5 -> 6
- net /matrix/col6: track 72.6 -> 88.6 mm
- net /led/lcol1: track 197.0 -> 182.3 mm
- net Net-(D0:7-Pad2): track 20.3 -> 9.53 mm
- net /matrix/col7: track 131.4 -> 122.5 mm
- net /led/lrow0: track 27.2 -> 22.0 mm
- net Net-(D0:5-Pad2): track 20.2 -> 23.3 mm
- net /matrix/row0: track 341.5 -> 343.8 mm
- net /led/lrow1: track 27.0 -> 25.7 mm
- net /matrix/row1: track 291.6 -> 292.5 mm, vias 1 -> 3

Commit message: adding prototype for revision 3: with more support for other layouts
Parts:
- added L1:0/1: LED, lib:CHERRY_MX_LED, F.Cu at (98.2, 126.8)
- added L1:12/13: LED, lib:CHERRY_MX_LED, F.Cu at (326.8, 126.8)
- added S1:0/1: SW_PUSH, lib:CHERRY_PCB_200H, F.Cu at (98.2, 126.8)
- added S1:12/13: SW_PUSH, lib:CHERRY_PCB_200H, F.Cu at (326.8, 126.8)
- moved R10 21.7 mm to (211.5, 135.0)
- moved U2 15.8 mm to (212.5, 117.0)
- moved C9 14.2 mm to (226.0, 116.0), turned to 270 degrees
- moved C10 13.0 mm to (199.0, 116.5), turned to 90 degrees
- moved R9 11.0 mm to (192.5, 121.0), turned to 90 degrees
Connections:
- L1:0 pad 1: Net-(L1:0-Pad1) -> Net-(L0:0-Pad1)
- L1:1 pad 1: Net-(L1:0-Pad1) -> Net-(L0:0-Pad1)
- L1:10 pad 1: Net-(L1:0-Pad1) -> Net-(L0:0-Pad1)
- L1:11 pad 1: Net-(L1:0-Pad1) -> Net-(L0:0-Pad1)
- L1:12 pad 1: Net-(L1:0-Pad1) -> Net-(L0:0-Pad1)
- L1:13 pad 1: Net-(L1:0-Pad1) -> Net-(L0:0-Pad1)
- L1:2 pad 1: Net-(L1:0-Pad1) -> Net-(L0:0-Pad1)
- L1:3 pad 1: Net-(L1:0-Pad1) -> Net-(L0:0-Pad1)
- L1:4 pad 1: Net-(L1:0-Pad1) -> Net-(L0:0-Pad1)
- L1:5 pad 1: Net-(L1:0-Pad1) -> Net-(L0:0-Pad1)
- L1:6 pad 1: Net-(L1:0-Pad1) -> Net-(L0:0-Pad1)
- L1:7 pad 1: Net-(L1:0-Pad1) -> Net-(L0:0-Pad1)
- L1:8 pad 1: Net-(L1:0-Pad1) -> Net-(L0:0-Pad1)
- L1:9 pad 1: Net-(L1:0-Pad1) -> Net-(L0:0-Pad1)
- R9 pad 1: Net-(L1:0-Pad1) -> Net-(L0:0-Pad1)
- S1:0 pad 1: /matrix/row1 -> /matrix/row0
- S1:1 pad 1: /matrix/row1 -> /matrix/row0
- S1:10 pad 1: /matrix/row1 -> /matrix/row0
- S1:11 pad 1: /matrix/row1 -> /matrix/row0
- S1:12 pad 1: /matrix/row1 -> /matrix/row0
- S1:13 pad 1: /matrix/row1 -> /matrix/row0
- S1:2 pad 1: /matrix/row1 -> /matrix/row0
- S1:3 pad 1: /matrix/row1 -> /matrix/row0
- S1:4 pad 1: /matrix/row1 -> /matrix/row0
- S1:5 pad 1: /matrix/row1 -> /matrix/row0
- S1:6 pad 1: /matrix/row1 -> /matrix/row0
- S1:7 pad 1: /matrix/row1 -> /matrix/row0
- S1:8 pad 1: /matrix/row1 -> /matrix/row0
- S1:9 pad 1: /matrix/row1 -> /matrix/row0
- U1 pad 26: /matrix/row1 -> /matrix/row0
Routing:
- net /matrix/row0: track 343.8 -> 0.00 mm, vias 2 -> 0
- net Net-(L0:0-Pad1): track 307.4 -> 0.00 mm, vias 2 -> 0
- net Net-(L4:0-Pad1): track 295.0 -> 0.00 mm, vias 2 -> 0
- net /matrix/row1: track 292.5 -> 0.00 mm, vias 3 -> 0
- net /matrix/row4: track 280.8 -> 0.00 mm
- net Net-(L3:0-Pad1): track 278.3 -> 0.00 mm, vias 3 -> 0
- net Net-(L2:0-Pad1): track 276.3 -> 0.00 mm
- net Net-(L1:0-Pad1): track 270.6 -> 0.00 mm
- net /matrix/row3: track 268.8 -> 0.00 mm, vias 1 -> 0
- net /matrix/row2: track 264.8 -> 0.00 mm, vias 4 -> 0
- net GND: track 218.3 -> 0.00 mm, vias 14 -> 0
- net /matrix/col13: track 207.8 -> 0.00 mm, vias 2 -> 0
- net /led/lcol0: track 207.4 -> 0.00 mm, vias 1 -> 0
- net /matrix/col0: track 202.9 -> 0.00 mm, vias 2 -> 0
- net /led/lcol13: track 202.5 -> 0.00 mm, vias 1 -> 0
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
Commit message: submitting quote for case and cover
Parts:
- M1, M2, M3, M4: footprint Mounting_Holes:MountingHole_4mm -> Mounting_Holes:MountingHole_6.4mm_M6
Changed lines of the file:
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@@
     (links 450)
     (no_connects 446)
-    (area 79.924999 60.674999 345.075001 154.825001)
+    (area 79.000799 44.15 360.65 158.929566)
     (thickness 1.6)
     (drawings 46)
@@
     )
   )
-  (module Mounting_Holes:MountingHole_4mm (layer F.Cu)
-    (at 117.5 117.24)
-    (descr "Mounting Hole 4mm, no annular")
-    (tags "mounting hole 4mm no annular")
-    (fp_text reference M3 (at 0 -5) (layer F.SilkS)
-      (effects (font (size 1 1) (thickness 0.15)))
-    )
-    (fp_text value MountingHole_4mm (at 0 5) (layer F.Fab)
-      (effects (font (size 1 1) (thickness 0.15)))
-    )
-    (fp_circle (center 0 0) (end 4 0) (layer Cmts.User) (width 0.15))
-    (fp_circle (center 0 0) (end 4.25 0) (layer F.CrtYd) (width 0.05))
-    (pad 1 np_thru_hole circle (at 0 0) (size 4 4) (drill 4) (layers *.Cu *.Mask))
-  )
-  (module Mounting_Holes:MountingHole_4mm (layer F.Cu)
-    (at 155.5 79.25)
-    (descr "Mounting Hole 4mm, no annular")
-    (tags "mounting hole 4mm no annular")
-    (fp_text reference M4 (at 0 -5) (layer F.SilkS)
-      (effects (font (size 1 1) (thickness 0.15)))
-    )
-    (fp_text value MountingHole_4mm (at 0 5) (layer F.Fab)
-      (effects (font (size 1 1) (thickness 0.15)))
-    )
-    (fp_circle (center 0 0) (end 4 0) (layer Cmts.User) (width 0.15))
-    (fp_circle (center 0 0) (end 4.25 0) (layer F.CrtYd) (width 0.05))
-    (pad 1 np_thru_hole circle (at 0 0) (size 4 4) (drill 4) (layers *.Cu *.Mask))
-  )
-  (module Mounting_Holes:MountingHole_4mm (layer F.Cu)
-    (at 269.5 136.25)
-    (descr "Mounting Hole 4mm, no annular")
-    (tags "mounting hole 4mm no annular")
-    (fp_text reference M1 (at 0 -5) (layer F.SilkS)
-      (effects (font (size 1 1) (thickness 0.15)))
-    )
-    (fp_text value MountingHole_4mm (at 0 5) (layer F.Fab)
-      (effects (font (size 1 1) (thickness 0.15)))
-    )
-    (fp_circle (center 0 0) (end 4 0) (layer Cmts.User) (width 0.15))
-    (fp_circle (center 0 0) (end 4.25 0) (layer F.CrtYd) (width 0.05))
-    (pad 1 np_thru_hole circle (at 0 0) (size 4 4) (drill 4) (layers *.Cu *.Mask))
-  )
-  (module Mounting_Holes:MountingHole_4mm (layer F.Cu)
-    (at 307.5 98.25)
-    (descr "Mounting Hole 4mm, no annular")
-    (tags "mounting hole 4mm no annular")
-    (fp_text reference M2 (at 0 -5) (layer F.SilkS)
-      (effects (font (size 1 1) (thickness 0.15)))
-    )
-    (fp_text value MountingHole_4mm (at 0 5) (layer F.Fab)
-      (effects (font (size 1 1) (thickness 0.15)))
-    )
-    (fp_circle (center 0 0) (end 4 0) (layer Cmts.User) (width 0.15))
-    (fp_circle (center 0 0) (end 4.25 0) (layer F.CrtYd) (width 0.05))
-    (pad 1 np_thru_hole circle (at 0 0) (size 4 4) (drill 4) (layers *.Cu *.Mask))
-  )
   (module .pretty:racc1 (layer B.Cu)
     (at 212.35 147.7 180)
@@
     )
   )
+  (module Mounting_Holes:MountingHole_6.4mm_M6 (layer F.Cu)
+    (at 117.5 117.24)
+    (descr "Mounting Hole 6.4mm, no annular, M6")
+    (tags "mounting hole 6.4mm no annular m6")
+    (fp_text reference M3 (at 0 -7.4) (layer F.SilkS)
+      (effects (font (size 1 1) (thickness 0.15)))
+    )
+    (fp_text value MountingHole_4mm (at 0 7.4) (layer F.Fab)
+      (effects (font (size 1 1) (thickness 0.15)))
+    )
+    (fp_circle (center 0 0) (end 6.4 0) (layer Cmts.User) (width 0.15))
+    (fp_circle (center 0 0) (end 6.65 0) (layer F.CrtYd) (width 0.05))
+    (pad 1 np_thru_hole circle (at 0 0) (size 6.4 6.4) (drill 6.4) (layers *.Cu *.Mask))
+  )
+  (module Mounting_Holes:MountingHole_6.4mm_M6 (layer F.Cu)
+    (at 155.5 79.25)
+    (descr "Mounting Hole 6.4mm, no annular, M6")
+    (tags "mounting hole 6.4mm no annular m6")
+    (fp_text reference M4 (at 0 -7.4) (layer F.SilkS)
+      (effects (font (size 1 1) (thickness 0.15)))
+    )
+    (fp_text value MountingHole_4mm (at 0 7.4) (layer F.Fab)
+      (effects (font (size 1 1) (thickness 0.15)))
+    )
+    (fp_circle (center 0 0) (end 6.4 0) (layer Cmts.User) (width 0.15))
+    (fp_circle (center 0 0) (end 6.65 0) (layer F.CrtYd) (width 0.05))
+    (pad 1 np_thru_hole circle (at 0 0) (size 6.4 6.4) (drill 6.4) (layers *.Cu *.Mask))
+  )
+  (module Mounting_Holes:MountingHole_6.4mm_M6 (layer F.Cu)
+    (at 269.5 136.25)
+    (descr "Mounting Hole 6.4mm, no annular, M6")
+    (tags "mounting hole 6.4mm no annular m6")
+    (fp_text reference M1 (at 0 -7.4) (layer F.SilkS)
+      (effects (font (size 1 1) (thickness 0.15)))
+    )
+    (fp_text value MountingHole_4mm (at 0 7.4) (layer F.Fab)
+      (effects (font (size 1 1) (thickness 0.15)))
+    )
+    (fp_circle (center 0 0) (end 6.4 0) (layer Cmts.User) (width 0.15))
+    (fp_circle (center 0 0) (end 6.65 0) (layer F.CrtYd) (width 0.05))
+    (pad 1 np_thru_hole circle (at 0 0) (size 6.4 6.4) (drill 6.4) (layers *.Cu *.Mask))
+  )
+  (module Mounting_Holes:MountingHole_6.4mm_M6 (layer F.Cu)
+    (at 307.5 98.25)
+    (descr "Mounting Hole 6.4mm, no annular, M6")
+    (tags "mounting hole 6.4mm no annular m6")
+    (fp_text reference M2 (at 0 -7.4) (layer F.SilkS)
+      (effects (font (size 1 1) (thickness 0.15)))
+    )
+    (fp_text value MountingHole_4mm (at 0 7.4) (layer F.Fab)
+      (effects (font (size 1 1) (thickness 0.15)))
+    )
+    (fp_circle (center 0 0) (end 6.4 0) (layer Cmts.User) (width 0.15))
+    (fp_circle (center 0 0) (end 6.65 0) (layer F.CrtYd) (width 0.05))
+    (pad 1 np_thru_hole circle (at 0 0) (size 6.4 6.4) (drill 6.4) (layers *.Cu *.Mask))
+  )
   (dimension 132.5 (width 0.3) (layer Cmts.User)
